File: eagle/usb-eeprom.brd (EAGLE design)
At the start: 82.2 x 22.9 mm, 13 parts, among them J1 USBA, U1 PIC18F45K50-I/PT

Commit message: Upgrade to EAGLE v6.6; update formatting
Parts:
- LOGO: value OSHW -> (none)
- renumbered U$1 to LOGO
Changed lines of the file:
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@@
 <?xml version="1.0" encoding="utf-8"?>
 <!DOCTYPE eagle SYSTEM "eagle.dtd">
-<eagle version="6.5.0">
+<eagle version="6.6.0">
 <drawing>
 <settings>
@@
 <setting verticaltext="up"/>
 </settings>
-<grid distance="0.025" unitdist="inch" unit="inch" style="lines" multiple="1" display="yes" altdistance="0.025" altunitdist="inch" altunit="inch"/>
+<grid distance="0.05" unitdist="inch" unit="inch" style="lines" multiple="1" display="yes" altdistance="0.025" altunitdist="inch" altunit="inch"/>
 <layers>
 <layer number="1" name="Top" color="4" fill="1" visible="yes" active="yes"/>
@@
 </autorouter>
 <elements>
-<element name="XU1" library="usb-eeprom" package="ZIF28" value="28CXXX-ZIF" x="55.3085" y="11.43" smashed="yes">
+<element name="XU1" library="usb-eeprom" package="ZIF28" value="28CXXX-ZIF" x="55.3085" y="11.43" locked="yes" smashed="yes">
 <attribute name="MOUSER_PN" value="517-228-1371-00" x="95.9485" y="-1.27" size="1.778" layer="27" display="off"/>
 <attribute name="MFG" value="3M" x="95.9485" y="-1.27" size="1.778" layer="27" display="off"/>
@@
 <attribute name="MFG_PN" value="228-1371-00-0602J" x="95.9485" y="-1.27" size="1.778" layer="27" display="off"/>
 <attribute name="NAME" x="31.75" y="1.27" size="1.27" layer="25" font="vector" align="center-right"/>
-<attribute name="VALUE" x="55.3085" y="11.43" size="1.27" layer="27" font="vector" align="center"/>
-</element>
-<element name="ICSP" library="usb-eeprom" package="ICSP" value="ICSP" x="21.59" y="20.955" smashed="yes">
+</element>
+<element name="ICSP" library="usb-eeprom" package="ICSP" value="ICSP" x="21.59" y="20.955" locked="yes" smashed="yes">
 <attribute name="NAME" x="29.21" y="19.05" size="1.27" layer="25" font="vector" align="top-right"/>
 </element>
-<element name="J1" library="usb-eeprom" package="USBA" value="USBA" x="2.9972" y="11.43" smashed="yes">
+<element name="J1" library="usb-eeprom" package="USBA" value="USBA" x="2.9972" y="11.43" locked="yes" smashed="yes">
 <attribute name="MOUSER_PN" value="538-48037-0001" x="41.0972" y="-20.32" size="1.778" layer="27" display="off"/>
 <attribute name="MFG" value="Molex" x="41.0972" y="-20.32" size="1.778" layer="27" display="off"/>
@@
 <attribute name="NAME" x="5.0927" y="17.78" size="1.27" layer="25" font="vector" align="top-left"/>
 </element>
-<element name="U1" library="usb-eeprom" package="TQFP44" value="PIC18F45K50-I/PT" x="21.59" y="11.43" smashed="yes" rot="R225">
+<element name="U1" library="usb-eeprom" package="TQFP44" value="PIC18F45K50-I/PT" x="21.59" y="11.43" locked="yes" smashed="yes" rot="R225">
 <attribute name="MOUSER_PN" value="579-PIC18F45K50-I/PT" x="-17.0251" y="17.71618125" size="1.778" layer="27" rot="R225" display="off"/>
 <attribute name="MFG" value="Microchip Technology" x="-17.0251" y="17.71618125" size="1.778" layer="27" rot="R225" display="off"/>
@@
 <attribute name="NAME" x="15.875" y="5.715" size="1.27" layer="25" font="vector" align="center"/>
 </element>
-<element name="R2" library="rcl" package="R0805" value="10K" x="10.16" y="16.51" smashed="yes" rot="R180">
+<element name="R2" library="rcl" package="R0805" value="10K" x="10.16" y="16.51" locked="yes" smashed="yes" rot="R180">
 <attribute name="MOUSER_PN" value="71-CRCW080510K0FKEB" x="-35.56" y="60.96" size="1.778" layer="27" rot="R180" display="off"/>
 <attribute name="MFG" value="Vishay" x="-35.56" y="60.96" size="1.778" layer="27" rot="R180" display="off"/>
@@
 <attribute name="NAME" x="10.16" y="15.24" size="0.762" layer="25" font="vector" align="top-center"/>
 </element>
-<element name="C4" library="rcl" package="C0805" value=".22uF" x="27.305" y="5.715" smashed="yes" rot="MR135">
+<element name="C4" library="rcl" package="C0805" value=".22uF" x="27.305" y="5.715" locked="yes" smashed="yes" rot="MR135">
 <attribute name="MOUSER_PN" value="77-VJ0805Y224KXJTBC" x="24.610921875" y="65.882715625" size="1.778" layer="28" rot="MR135" display="off"/>
 <attribute name="MFG" value="Vishay" x="24.610921875" y="65.882715625" size="1.778" layer="28" rot="MR135" display="off"/>
@@
 <attribute name="NAME" x="29.21" y="3.81" size="0.762" layer="26" font="vector" rot="MR0"/>
 </element>
-<element name="R3" library="rcl" package="R0805" value="10K" x="10.16" y="11.43" smashed="yes" rot="R180">
+<element name="R3" library="rcl" package="R0805" value="10K" x="10.16" y="11.43" locked="yes" smashed="yes" rot="R180">
 <attribute name="MOUSER_PN" value="71-CRCW080510K0FKEB" x="-40.64" y="55.88" size="1.778" layer="27" rot="R180" display="off"/>
 <attribute name="MFG" value="Vishay" x="-40.64" y="55.88" size="1.778" layer="27" rot="R180" display="off"/>
@@
 <attribute name="NAME" x="10.16" y="10.16" size="0.762" layer="25" font="vector" align="top-center"/>
 </element>
-<element name="R1" library="rcl" package="R0805" value="100" x="10.16" y="20.955" smashed="yes">
+<element name="R1" library="rcl" package="R0805" value="100" x="10.16" y="20.955" locked="yes" smashed="yes">
 <attribute name="MOUSER_PN" value="71-CRCW0805-100-E3" x="66.04" y="-23.495" size="1.778" layer="27" display="off"/>
 <attribute name="MFG" value="Vishay" x="66.04" y="-23.495" size="1.778" layer="27" display="off"/>
@@
 <attribute name="NAME" x="4.445" y="19.685" size="0.762" layer="25" font="vector" align="top-center"/>
 </element>
-<element name="C1" library="rcl" package="C0805" value=".1uF" x="34.925" y="19.05" smashed="yes" rot="MR0">
+<element name="C1" library="rcl" package="C0805" value=".1uF" x="34.925" y="19.05" locked="yes" smashed="yes" rot="MR0">
 <attribute name="MOUSER_PN" value="77-VJ0805Y104KXJCBC" x="18.415" y="-34.29" size="1.778" layer="28" rot="MR0" display="off"/>
 <attribute name="MFG" value="Vishay" x="18.415" y="-34.29" size="1.778" layer="28" rot="MR0" display="off"/>
@@
 <attribute name="NAME" x="34.925" y="20.32" size="0.762" layer="26" font="vector" rot="MR0" align="bottom-center"/>
 </element>
-<element name="C2" library="rcl" package="C0805" value=".1uF" x="15.875" y="5.715" smashed="yes" rot="MR225">
+<element name="C2" library="rcl" package="C0805" value=".1uF" x="15.875" y="5.715" locked="yes" smashed="yes" rot="MR225">
 <attribute name="MOUSER_PN" value="77-VJ0805Y104KXJCBC" x="68.858509375" y="28.1656375" size="1.778" layer="28" rot="MR225" display="off"/>
 <attribute name="MFG" value="Vishay" x="68.858509375" y="28.1656375" size="1.778" layer="28" rot="MR225" display="off"/>
@@
 <attribute name="NAME" x="13.97" y="3.81" size="0.762" layer="26" font="vector" rot="MR0" align="bottom-right"/>
 </element>
-<element name="C3" library="rcl" package="C0805" value=".1uF" x="27.305" y="17.145" smashed="yes" rot="MR225">
+<element name="C3" library="rcl" package="C0805" value=".1uF" x="27.305" y="17.145" locked="yes" smashed="yes" rot="MR225">
 <attribute name="MOUSER_PN" value="77-VJ0805Y104KXJCBC" x="83.8806125" y="36.0035375" size="1.778" layer="28" rot="MR225" display="off"/>
 <attribute name="MFG" value="Vishay" x="83.8806125" y="36.0035375" size="1.778" layer="28" rot="MR225" display="off"/>
@@
 <attribute name="NAME" x="29.21" y="19.05" size="0.762" layer="26" font="vector" rot="MR0" align="top-left"/>
 </element>
-<element name="U$1" library="usb-eeprom" package="OSHW" value="OSHW" x="7.3025" y="3.683"/>
+<element name="LOGO" library="usb-eeprom" package="OSHW" value="" x="7.3025" y="3.683" locked="yes"/>
 </elements>
 <signals>
@@
 <contactref element="C2" pad="2"/>
 <contactref element="C3" pad="2"/>
-<polygon width="0.4064" layer="16">
+<polygon width="0.1524" layer="16">
 <vertex x="82.2325" y="21.59"/>
 <vertex x="82.2325" y="1.27" curve="-90"/>
